File: finch_pack.sch (EAGLE design)
At the start: 5 parts

Commit message: schematic file
Parts:
- removed FHM-02PG: FHM-02PG, fujikura-fhm:FHM-02PG
- added FHM-02PGR: FHM-02PGR, fujikura-fhm:FHM-02PGR
Connections:
- net GND: now also FHM-02PGR.V-; no longer FHM-02PG.V-
- net N$1: now also FHM-02PGR.VO+; no longer FHM-02PG.VO+
- net N$2: now also FHM-02PGR.VO-@1, FHM-02PGR.VO-@6; no longer FHM-02PG.VO-@1, FHM-02PG.VO-@6
- net N$4: now also FHM-02PGR.V+; no longer FHM-02PG.V+
Changed lines of the file:
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@@
 </classes>
 <parts>
-<part name="FHM-02PG" library="fujikura-fhm" deviceset="FHM-02PG" device=""/>
+<part name="FHM-02PGR" library="fujikura-fhm" deviceset="FHM-02PGR" device=""/>
 <part name="INA122UA" library="texas-ina" deviceset="INA122UA" device=""/>
 <part name="R1" library="rcl" library_urn="urn:adsk.eagle:library:334" deviceset="R-US_" device="0309/10" package3d_urn="urn:adsk.eagle:package:23567/2"/>
@@
 </plain>
 <instances>
-<instance part="FHM-02PG" gate="G$1" x="22.86" y="15.24" smashed="yes" rot="R90">
+<instance part="FHM-02PGR" gate="G$1" x="22.86" y="15.24" smashed="yes" rot="R90">
 <attribute name="NAME" x="10.16" y="10.16" size="1.27" layer="95" rot="R90"/>
 <attribute name="VALUE" x="38.1" y="10.16" size="1.27" layer="95" rot="R90"/>
@@
 <wire x1="30.48" y1="30.48" x2="46.3" y2="30.48" width="0.1524" layer="91"/>
 <wire x1="46.3" y1="30.48" x2="46.3" y2="20.32" width="0.1524" layer="91"/>
-<pinref part="FHM-02PG" gate="G$1" pin="VO+"/>
+<pinref part="FHM-02PGR" gate="G$1" pin="VO+"/>
 <junction x="30.48" y="30.48"/>
 <pinref part="INA122UA" gate="G$1" pin="VIN+"/>
@@
 <wire x1="7.62" y1="-5.08" x2="15.24" y2="-5.08" width="0.1524" layer="91"/>
 <junction x="15.24" y="-5.08"/>
-<pinref part="FHM-02PG" gate="G$1" pin="VO-@1"/>
+<pinref part="FHM-02PGR" gate="G$1" pin="VO-@1"/>
 <junction x="15.24" y="30.48"/>
-<pinref part="FHM-02PG" gate="G$1" pin="VO-@6"/>
+<pinref part="FHM-02PGR" gate="G$1" pin="VO-@6"/>
 <pinref part="INA122UA" gate="G$1" pin="VIN-"/>
 </segment>
@@
 <wire x1="22.86" y1="0" x2="22.86" y2="-5.08" width="0.1524" layer="91"/>
 <wire x1="22.86" y1="-5.08" x2="50.8" y2="-5.08" width="0.1524" layer="91"/>
-<pinref part="FHM-02PG" gate="G$1" pin="V-"/>
+<pinref part="FHM-02PGR" gate="G$1" pin="V-"/>
 <pinref part="INA122UA" gate="G$1" pin="V-"/>
 <pinref part="INA122UA" gate="G$1" pin="REF"/>
@@
 <net name="N$4" class="0">
 <segment>
-<pinref part="FHM-02PG" gate="G$1" pin="V+"/>
+<pinref part="FHM-02PGR" gate="G$1" pin="V+"/>
 <wire x1="22.86" y1="30.48" x2="22.86" y2="38.1" width="0.1524" layer="91"/>
 <pinref part="R2" gate="G$1" pin="2"/>
