File: finch_pack.sch (EAGLE design)
At the start: 5 parts

Commit message: schematic file
Connections:
- removed net N$4: FHM-02PGR.V+, R2.2
- new net N$3: FHM-02PGR.VO-@1, R2.1
- net N$2: now also R2.2; no longer FHM-02PGR.VO-@1
- net V+: now also FHM-02PGR.V+; no longer R2.1
Other:
- moved on the sheet: R2
Changed lines of the file:
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@@
 <instances>
 <instance part="FHM-02PGR" gate="G$1" x="22.86" y="15.24" smashed="yes" rot="R90">
-<attribute name="NAME" x="10.16" y="10.16" size="1.27" layer="95" rot="R90"/>
+<attribute name="NAME" x="20.32" y="10.16" size="1.27" layer="95" rot="R90"/>
 <attribute name="VALUE" x="38.1" y="10.16" size="1.27" layer="95" rot="R90"/>
 </instance>
@@
 <attribute name="VALUE" x="39.878" y="16.51" size="1.778" layer="96" rot="R270"/>
 </instance>
-<instance part="R2" gate="G$1" x="33.02" y="38.1" smashed="yes" rot="R180">
-<attribute name="NAME" x="36.83" y="36.6014" size="1.778" layer="95" rot="R180"/>
-<attribute name="VALUE" x="36.83" y="41.402" size="1.778" layer="96" rot="R180"/>
+<instance part="R2" gate="G$1" x="7.62" y="12.7" smashed="yes" rot="R270">
+<attribute name="NAME" x="9.1186" y="16.51" size="1.778" layer="95" rot="R270"/>
+<attribute name="VALUE" x="4.318" y="16.51" size="1.778" layer="96" rot="R270"/>
 </instance>
 <instance part="CONNECTOR" gate="A" x="83.82" y="40.64" smashed="yes">
@@
 <wire x1="43.18" y1="-10.16" x2="43.18" y2="5.08" width="0.1524" layer="91"/>
 <wire x1="43.18" y1="5.08" x2="46.3" y2="5.08" width="0.1524" layer="91"/>
-<wire x1="15.24" y1="30.48" x2="7.62" y2="30.48" width="0.1524" layer="91"/>
-<wire x1="7.62" y1="30.48" x2="7.62" y2="-5.08" width="0.1524" layer="91"/>
 <wire x1="7.62" y1="-5.08" x2="15.24" y2="-5.08" width="0.1524" layer="91"/>
 <junction x="15.24" y="-5.08"/>
-<pinref part="FHM-02PGR" gate="G$1" pin="VO-@1"/>
-<junction x="15.24" y="30.48"/>
 <pinref part="FHM-02PGR" gate="G$1" pin="VO-@6"/>
 <pinref part="INA122UA" gate="G$1" pin="VIN-"/>
+<wire x1="7.62" y1="7.62" x2="7.62" y2="-5.08" width="0.1524" layer="91"/>
+<pinref part="R2" gate="G$1" pin="2"/>
 </segment>
 </net>
@@
 </segment>
 </net>
-<net name="N$4" class="0">
-<segment>
-<pinref part="FHM-02PGR" gate="G$1" pin="V+"/>
-<wire x1="22.86" y1="30.48" x2="22.86" y2="38.1" width="0.1524" layer="91"/>
-<pinref part="R2" gate="G$1" pin="2"/>
-<wire x1="22.86" y1="38.1" x2="27.94" y2="38.1" width="0.1524" layer="91"/>
-</segment>
-</net>
 <net name="V+" class="0">
 <segment>
 <pinref part="INA122UA" gate="G$1" pin="V+"/>
+<wire x1="22.86" y1="38.1" x2="43.18" y2="38.1" width="0.1524" layer="91"/>
 <wire x1="43.18" y1="38.1" x2="62.54" y2="38.1" width="0.1524" layer="91"/>
 <wire x1="62.54" y1="38.1" x2="62.54" y2="23.36" width="0.1524" layer="91"/>
+<pinref part="FHM-02PGR" gate="G$1" pin="V+"/>
+<wire x1="22.86" y1="30.48" x2="22.86" y2="38.1" width="0.1524" layer="91"/>
 <pinref part="CONNECTOR" gate="A" pin="1"/>
-<wire x1="43.18" y1="38.1" x2="43.18" y2="43.18" width="0.1524" layer="91"/>
 <wire x1="43.18" y1="43.18" x2="81.28" y2="43.18" width="0.1524" layer="91"/>
-<pinref part="R2" gate="G$1" pin="1"/>
-<wire x1="38.1" y1="38.1" x2="43.18" y2="38.1" width="0.1524" layer="91"/>
+<label x="86.36" y="43.18" size="1.778" layer="95"/>
+<wire x1="43.18" y1="43.18" x2="43.18" y2="38.1" width="0.1524" layer="91"/>
 <junction x="43.18" y="38.1"/>
-<label x="86.36" y="43.18" size="1.778" layer="95"/>
 </segment>
 </net>
@@
 </segment>
 </net>
+<net name="N$3" class="0">
+<segment>
+<pinref part="FHM-02PGR" gate="G$1" pin="VO-@1"/>
+<junction x="15.24" y="30.48"/>
+<wire x1="15.24" y1="30.48" x2="7.62" y2="30.48" width="0.1524" layer="91"/>
+<wire x1="7.62" y1="30.48" x2="7.62" y2="17.78" width="0.1524" layer="91"/>
+<pinref part="R2" gate="G$1" pin="1"/>
+</segment>
+</net>

Commit message: schematic file
Parts:
- R1: value (none) -> 2200
- R2: value (none) -> 100
Changed lines of the file:
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@@
 <part name="FHM-02PGR" library="fujikura-fhm" deviceset="FHM-02PGR" device=""/>
 <part name="INA122UA" library="texas-ina" deviceset="INA122UA" device=""/>
-<part name="R1" library="rcl" library_urn="urn:adsk.eagle:library:334" deviceset="R-US_" device="0309/10" package3d_urn="urn:adsk.eagle:package:23567/2"/>
-<part name="R2" library="rcl" library_urn="urn:adsk.eagle:library:334" deviceset="R-US_" device="0309/10" package3d_urn="urn:adsk.eagle:package:23567/2"/>
+<part name="R1" library="rcl" library_urn="urn:adsk.eagle:library:334" deviceset="R-US_" device="0309/10" package3d_urn="urn:adsk.eagle:package:23567/2" value="2200"/>
+<part name="R2" library="rcl" library_urn="urn:adsk.eagle:library:334" deviceset="R-US_" device="0309/10" package3d_urn="urn:adsk.eagle:package:23567/2" value="100"/>
 <part name="CONNECTOR" library="pinhead" library_urn="urn:adsk.eagle:library:325" deviceset="PINHD-1X3" device="" package3d_urn="urn:adsk.eagle:package:22458/2"/>
 </parts>
