File: finch_pack.brd (EAGLE design)
At the start: 14.6 x 28.3 mm, 5 parts

Commit message: board file
Parts:
- FHM-02PGR: value FHM-02PG -> FHM-02PGR
- renumbered FHM-02PG to FHM-02PGR
Changed lines of the file:
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@@
 </autorouter>
 <elements>
-<element name="FHM-02PG" library="fujikura-fhm" package="FHM-02PG" value="FHM-02PG" x="7.482109375" y="19.67463125" smashed="yes">
+<element name="FHM-02PGR" library="fujikura-fhm" package="FHM-02PG" value="FHM-02PGR" x="7.482109375" y="19.67463125" smashed="yes">
 <attribute name="NAME" x="4.8442" y="16.611578125" size="0.254" layer="32" display="off"/>
 <attribute name="VALUE" x="5.80945625" y="17.18913125" size="0.4064" layer="21"/>
@@
 <signals>
 <signal name="N$1">
-<contactref element="FHM-02PG" pad="3"/>
+<contactref element="FHM-02PGR" pad="3"/>
 <contactref element="INA122UA" pad="3"/>
 <wire x1="7.032625" y1="12.99173125" x2="13.444609375" y2="12.99173125" width="0.1524" layer="1"/>
@@
 </signal>
 <signal name="N$2">
-<contactref element="FHM-02PG" pad="1"/>
-<contactref element="FHM-02PG" pad="6"/>
+<contactref element="FHM-02PGR" pad="1"/>
+<contactref element="FHM-02PGR" pad="6"/>
 <contactref element="INA122UA" pad="2"/>
 <wire x1="2.402109375" y1="22.21463125" x2="3.59519375" y2="21.021546875" width="0.1524" layer="1"/>
@@
 </signal>
 <signal name="GND">
-<contactref element="FHM-02PG" pad="5"/>
+<contactref element="FHM-02PGR" pad="5"/>
 <contactref element="INA122UA" pad="4"/>
 <contactref element="INA122UA" pad="5"/>
@@
 <wire x1="2.402109375" y1="19.144275" x2="1.114040625" y2="17.85620625" width="0.1524" layer="16"/>
 <wire x1="1.114040625" y1="17.85620625" x2="1.114040625" y2="3.86304375" width="0.1524" layer="16"/>
-<wire x1="1.0958875" y1="10.547521875" x2="1.82549375" y2="9.817915625" width="0.1524" layer="1"/>
+<wire x1="1.82549375" y1="9.817915625" x2="1.0958875" y2="10.547521875" width="0.1524" layer="1"/>
 <wire x1="1.82549375" y1="9.817915625" x2="4.81986875" y2="9.817915625" width="0.1524" layer="1"/>
 </signal>
 <signal name="N$4">
-<contactref element="FHM-02PG" pad="2"/>
+<contactref element="FHM-02PGR" pad="2"/>
 <wire x1="12.435109375" y1="19.67463125" x2="12.435109375" y2="19.33058125" width="0.1524" layer="16"/>
 <wire x1="12.435109375" y1="19.33058125" x2="2.163228125" y2="9.0587" width="0.1524" layer="16"/>

Commit message: board file
Parts:
- FHM-02PGR: device fujikura-fhm:FHM-02PG -> fujikura-fhm:FHM-02PGR
Changed lines of the file:
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@@
 </autorouter>
 <elements>
-<element name="FHM-02PGR" library="fujikura-fhm" package="FHM-02PG" value="FHM-02PGR" x="7.482109375" y="19.67463125" smashed="yes">
+<element name="FHM-02PGR" library="fujikura-fhm" package="FHM-02PGR" value="FHM-02PGR" x="7.482109375" y="19.67463125" smashed="yes">
 <attribute name="NAME" x="4.8442" y="16.611578125" size="0.254" layer="32" display="off"/>
 <attribute name="VALUE" x="5.80945625" y="17.18913125" size="0.4064" layer="21"/>

Commit message: board file
Parts:
- moved R1 0.48 mm to (7.24, 25.9)
Connections:
- removed net N$4: FHM-02PGR.2, R2.2
- new net N$3: FHM-02PGR.1, R2.1
- net N$2: now also R2.2; no longer FHM-02PGR.1
- net V+: now also FHM-02PGR.2; no longer R2.1
Routing:
- net N$3: track 0.00 -> 18.5 mm
- net N$4: track 17.4 -> 0.00 mm
- net V+: track 15.0 -> 25.3 mm
- net GND: track 39.0 -> 32.5 mm
- net N$2: track 21.8 -> 18.1 mm
- net N$1: track 15.0 -> 12.5 mm
Other:
- board size 14.6 x 28.3 mm -> 14.7 x 28 mm

Commit message: board file
Parts:
- R1: value (none) -> 2200
- R2: value (none) -> 100
Changed lines of the file:
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@@
 <drawing>
 <settings>
-<setting alwaysvectorfont="yes"/>
+<setting alwaysvectorfont="no"/>
 <setting verticaltext="up"/>
 </settings>
@@
 <attribute name="VALUE" x="7.287884375" y="10.52328125" size="0.4064" layer="27" align="top-center"/>
 </element>
-<element name="R1" library="rcl" library_urn="urn:adsk.eagle:library:334" package="0309/10" package3d_urn="urn:adsk.eagle:package:23567/2" value="" x="7.242403125" y="25.862809375" smashed="yes" rot="MR180">
-<attribute name="NAME" x="3.602975" y="26.580146875" size="0.4064" layer="26" ratio="10" rot="MR180"/>
+<element name="R1" library="rcl" library_urn="urn:adsk.eagle:library:334" package="0309/10" package3d_urn="urn:adsk.eagle:package:23567/2" value="2200" x="7.242403125" y="25.862809375" smashed="yes" rot="MR180">
+<attribute name="NAME" x="10.329240625" y="25.403328125" size="0.4064" layer="26" ratio="10" rot="MR180"/>
 <attribute name="POPULARITY" value="0" x="7.242403125" y="25.862809375" size="1.778" layer="28" rot="MR180" display="off"/>
 <attribute name="SPICEPREFIX" value="R" x="7.242403125" y="25.862809375" size="1.778" layer="28" rot="MR180" display="off"/>
-<attribute name="VALUE" x="4.067403125" y="26.548609375" size="1.27" layer="28" ratio="10" rot="MR180"/>
-</element>
-<element name="R2" library="rcl" library_urn="urn:adsk.eagle:library:334" package="0309/10" package3d_urn="urn:adsk.eagle:package:23567/2" value="" x="7.243228125" y="6.551809375" smashed="yes" rot="MR0">
+<attribute name="VALUE" x="4.067403125" y="26.548609375" size="0.3048" layer="28" ratio="10" rot="MR180"/>
+</element>
+<element name="R2" library="rcl" library_urn="urn:adsk.eagle:library:334" package="0309/10" package3d_urn="urn:adsk.eagle:package:23567/2" value="100" x="7.243228125" y="6.551809375" smashed="yes" rot="MR0">
 <attribute name="NAME" x="11.02055" y="5.627446875" size="0.4064" layer="26" ratio="10" rot="MR0"/>
 <attribute name="POPULARITY" value="0" x="7.243228125" y="6.551809375" size="1.778" layer="28" rot="MR0" display="off"/>
 <attribute name="SPICEPREFIX" value="R" x="7.243228125" y="6.551809375" size="1.778" layer="28" rot="MR0" display="off"/>
-<attribute name="VALUE" x="10.418228125" y="5.866009375" size="1.27" layer="28" ratio="10" rot="MR0"/>
+<attribute name="VALUE" x="4.91491875" y="7.04283125" size="0.3048" layer="28" ratio="10" rot="MR0"/>
 </element>
 <element name="CONNECTOR" library="pinhead" library_urn="urn:adsk.eagle:library:325" package="1X03" package3d_urn="urn:adsk.eagle:package:22458/2" value="" x="7.15206875" y="2.6402625" smashed="yes" rot="R180">
@@
 <wire x1="3.59519375" y1="21.021546875" x2="3.59519375" y2="12.2426" width="0.1524" layer="1"/>
 <wire x1="3.59519375" y1="12.2426" x2="3.585228125" y2="12.232634375" width="0.1524" layer="1"/>
-<wire x1="3.585228125" y1="12.232634375" x2="4.577003125" y2="12.232634375" width="0.1524" layer="1"/>
-<wire x1="4.577003125" y1="12.232634375" x2="4.6945875" y2="12.232634375" width="0.1524" layer="1"/>
+<wire x1="3.585228125" y1="12.232634375" x2="4.6945875" y2="12.232634375" width="0.1524" layer="1"/>
 <wire x1="4.6945875" y1="12.232634375" x2="4.81986875" y2="12.357915625" width="0.1524" layer="1"/>
 <contactref element="R2" pad="2"/>
